File: _autosave-motor_control_design.kicad_sch (KiCad schematic)
At the start: 90 parts, among them J1 TYPE-C-31-M-12, J10 5V, J2 SWD, J3 VBAT, J4 GND, J5 FC_M/P, J6 Conn_01x06, J7 Conn_01x04_Pin, J8 Conn_01x06, J9 GND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

Commit message: ADR2
Put the 8th mosfet back, fixed all of ethans criteia
Changed lines of the file:
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@@
 		(at 67.31 95.25)
+	)
+	(bus_entry
+		(at 90.17 180.34)
+		(size 2.54 2.54)
+		(stroke
+			(width 0)
+			(type default)
+		)
 	)
 	(polyline
