File: _autosave-motor_control_design.kicad_pcb (KiCad board)
At the start: 4 copper layers, 57.1 x 58.8 mm, 113 parts, among them J1 TYPE-C-31-M-12, J2 SWD, J3 XT30UPB-F, J5 XT30UPB-M, J6 Conn_01x06, J7 Conn_01x04_Pin, J8 Conn_01x06, Q1 RF1S9540SM, Q10 2N7002, Q11 2N7002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

Commit message: BUILD files
Parts:
- D11, D13, D14, D18, D19, D21, D22, D23: footprint Diode_SMD:D_SOD-882 -> Diode_SMD:D_0402_1005Metric
- R25, R26: value 5.11k -> 5k
- R33: value 5.1k -> 5k
- moved J5 5.01 mm to (132.4, 66.9), turned to -140 degrees
- moved D19 0.55 mm to (161.0, 72.2)
- moved D21 0.45 mm to (133.5, 107.5)
- moved D18 0.19 mm to (162.1, 72.2)
Connections:
- J5 pad 1: GND -> +BATT
- J5 pad 2: +BATT -> GND
Routing:
- net /SCL: track 51.4 -> 52.5 mm
